File: electronics/mainBoard_kicad_independent_pumps/main_board_independent_pumps.kicad_pcb (KiCad board)
At the start: 2 copper layers, 127 x 93 mm, 32 parts, among them J1 A_lim, J10 5v, J11 24v, J12 Conn_01x04_Socket, J13 Conn_01x04_Socket, J2 B_lim, J3 Z_lim, J4 Conn_01x04_Socket, J5 Conn_01x04_Socket, J6 Conn_01x04_Socket, J7 Conn_01x04_Socket, J8 Conn_01x04_Socket, J9 Conn_01x04_Socket, SW1 SW_DPDT_x2

Commit message: prelim changes
Connections:
- 3b+header1 pad 1: unconnected-(3b+header1-5V-Pad1) -> +5V
- 3b+header1 pad 3: /logic_power -> +5V
Routing:
- net +5V: track 305.2 -> 324.4 mm
Changed lines of the file:
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@@
 			(layers "*.Cu" "*.Mask")
 			(remove_unused_layers no)
-			(net "unconnected-(3b+header1-5V-Pad1)")
+			(net "+5V")
 			(pinfunction "5V_1")
 			(pintype "output")
@@
 			(layers "*.Cu" "*.Mask")
 			(remove_unused_layers no)
-			(net "/logic_power")
+			(net "+5V")
 			(pinfunction "5V_3")
 			(pintype "output")
@@
 	)
 	(segment
+		(start 112.5 54)
+		(end 106.7 59.8)
+		(width 0.6)
+		(layer "F.Cu")
+		(net "+5V")
+	)
+	(segment
 		(start 142.631371 49.5)
 		(end 142.331371 49.8)
@@
 	)
 	(segment
+		(start 106.7 59.8)
+		(end 106.54 59.8)
+		(width 0.6)
+		(layer "F.Cu")
+		(net "+5V")
+	)
+	(segment
 		(start 192.35 83)
 		(end 184.5 83)
@@
 	)
 	(segment
+		(start 106.54 62.34)
+		(end 112.5 56.38)
+		(width 0.6)
+		(layer "B.Cu")
+		(net "+5V")
+	)
+	(segment
 		(start 153 98.5)
 		(end 155.41 96.09)
@@
 		(width 0.6)
 		(layer "B.Cu")
+		(net "+5V")
+	)
+	(segment
+		(start 112.5 56.38)
+		(end 112.5 54)
+		(width 0.6)
+		(layer "B.Cu")
